File: Thermometer.kicad_pcb (KiCad board)
At the start: 2 copper layers, 70 x 50 mm, 37 parts, among them J1 Conn_01x03_Socket, J2 Conn_01x03_Socket, J3 Conn_01x04, J4 USB_C_Receptacle_USB2.0_14P, J5 Conn_01x02, SW1 SW_Push, SW2 SW_Push, U1 ESP32-C6-WROOM-1, U2 HDC2080, U3 LM75B, U4 TLV75733PDBV, U5 TMP102xxDRL, U6 USBLC6-2SC6

Commit message: second commit
Parts:
- added REF**: MountingHole_3.2mm_M3_Pad_Via, MountingHole:MountingHole_3.2mm_M3_Pad_Via, F.Cu at (212.2, 81.9)
- added REF**: MountingHole_3.2mm_M3_Pad_Via, MountingHole:MountingHole_3.2mm_M3_Pad_Via, F.Cu at (212.0, 47.0)
- moved R3 17.9 mm to (183.8, 69.0)
- moved R2 17.2 mm to (180.2, 66.5)
- moved TP2 11.2 mm to (167.0, 78.8)
- moved J1 10.0 mm to (175.0, 46.3)
- moved J2 9.25 mm to (187.8, 46.3)
- moved R1 8.90 mm to (162.1, 82.5)
- moved J3 8.23 mm to (196.9, 45.5)
- moved SW1 8.19 mm to (167.8, 73.8)
- moved C1 7.42 mm to (165.3, 82.5)
- moved C2 6.05 mm to (160.8, 77.2)
- moved C3 5.52 mm to (161.0, 73.5)
- moved J5 3.07 mm to (203.0, 79.2)
- moved R7 2.15 mm to (204.2, 65.2), turned to 0 degrees
- moved C6 1.72 mm to (196.7, 73.5)
- moved TP4 1.12 mm to (194.0, 70.0)
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Routing:
- net +3.3V: track 0.00 -> 171.6 mm, vias 0 -> 4
- net /sda: track 0.00 -> 48.9 mm, vias 0 -> 2
- net /scl: track 0.00 -> 45.6 mm
- net /U0RXD: track 0.00 -> 41.7 mm
- net /GPIO18: track 0.00 -> 40.0 mm, vias 0 -> 2
- net /U0TXD: track 0.00 -> 37.6 mm
- net /GPIO19: track 0.00 -> 29.3 mm, vias 0 -> 2
- net VBUS: track 0.00 -> 29.1 mm
- net /GPIO3: track 0.00 -> 27.2 mm
- net Net-(U1-EN/CHIP_PU): track 0.00 -> 21.1 mm
- net Net-(D1-K): track 0.00 -> 18.6 mm
- net Net-(U1-GPIO9): track 0.00 -> 17.9 mm
- net /GPIO2: track 0.00 -> 16.7 mm
- net /GPIO20: track 0.00 -> 15.7 mm
- net /USB_D-: track 0.00 -> 8.55 mm
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- added copper zone on F.Cu, net GND
Other:
- board size 70 x 50 mm -> 63 x 50 mm
- rule pad_to_mask_clearance: 0.1 -> 0
