File: Thermometer.kicad_pcb (KiCad board)
At the start: 2 copper layers, 63 x 50 mm, 39 parts, among them J1 Conn_01x03_Socket, J2 Conn_01x03_Socket, J3 Conn_01x04, J4 USB_C_Receptacle_USB2.0_14P, J5 Conn_01x02, SW1 SW_Push, SW2 SW_Push, U1 ESP32-C6-WROOM-1, U2 HDC2080, U3 LM75B, U4 TLV75733PDBV, U5 TMP102xxDRL, U6 USBLC6-2SC6

Commit message: ajout des fichiers de production
Parts:
- C2: footprint Capacitor_SMD:C_1210_3225Metric -> Capacitor_SMD:C_1206_3216Metric
Routing:
- net +3.3V: track 171.6 -> 192.5 mm, vias 4 -> 6
- net Net-(J4-CC2): track 5.18 -> 5.75 mm
- net VBUS: track 29.1 -> 29.6 mm
- net GND: vias 34 -> 35
Other:
- board text added: "CornetPrisme"
- board text added: "Thermometer"

Commit message: changement de disposition
Parts:
- moved U2 32.4 mm to (214.8, 65.0), turned to 90 degrees
- moved U5 24.8 mm to (215.2, 71.2)
- moved C7 13.2 mm to (215.6, 60.0)
- moved R7 13.2 mm to (215.6, 58.5)
- moved U3 13.2 mm to (214.6, 55.2)
- moved TP3 8.31 mm to (188.8, 61.5)
- moved TP1 3.34 mm to (193.5, 57.2)
- moved REF** 2.11 mm to (212.0, 84.0)
- moved J5 1.77 mm to (202.7, 81.0)
- moved REF** 1.00 mm to (212.0, 46.0)
Routing:
- net GND: track 0.00 -> 75.8 mm, vias 35 -> 36
- net /GPIO20: track 15.7 -> 57.7 mm, vias 0 -> 2
- net /scl: track 45.9 -> 87.2 mm, vias 0 -> 4
- net /GPIO19: track 29.3 -> 62.5 mm
- net /sda: track 48.9 -> 79.0 mm, vias 2 -> 0
- net /GPIO18: track 40.0 -> 54.0 mm
- net +3.3V: track 192.5 -> 199.6 mm
Other:
- outline, holes or cut-outs redrawn
- board text added: "Thermometer 09/2026"
- board text added: "adiabatique™"
- board text removed: "Thermometer"

Commit message: Ajout image
Parts:
- added G***: LOGO, LOGO, B.Cu at (164.0, 78.5)
Other:
- board text added: "3.3V"
- board text added: "5V"
- board text added: "Boot"
- board text added: "GND"
- board text added: "HDC2080"
- board text added: "LM75"
- board text added: "RX"
- board text added: "Rst"
- board text added: "TMP102"
- board text added: "TX"
- board text added: "Victor Blain"
- board text added: "scl"
- board text added: "sda"

Commit message: changement fichiers production
Parts:
- U3: footprint Package_SO:TSSOP-8_3x3mm_P0.65mm -> Package_SO:SOIC-8_3.9x4.9mm_P1.27mm
- moved U3 1.17 mm to (215.2, 54.2)
Routing:
- net GND: track 75.8 -> 82.3 mm, vias 36 -> 34
- net +3.3V: track 199.6 -> 201.4 mm
- net /scl: track 87.2 -> 88.7 mm
- net /GPIO18: track 54.0 -> 55.0 mm
